File: KiCAD/ProdDeck/ProdDeck.kicad_sch (KiCad schematic)
At the start: 0 parts

Commit message: working?
Parts:
- added BATT_CONN1: BATT_CONN1, Connector_JST:JST_PH_S2B-PH-K_1x02_P2.00mm_Horizontal, symbol Connector_Generic:Conn_01x02
- added BOOT0: BOOT0, Button_Switch_SMD:SW_SPST_CK_RS282G05A3, symbol Switch:SW_Push
- added BT1: LiPo 3.7V 500mAh, symbol Device:Battery_Cell
- added C1, C10, C19, C3, C5, C6: 4u7, Capacitor_SMD:C_0603_1608Metric, symbol Device:C
- added C11, C12, C13, C14, C15, C18, C22, C4, C7, C8, C9: 100n, Capacitor_SMD:C_0402_1005Metric, symbol Device:C
- added C16, C17: 10p, Capacitor_SMD:C_0402_1005Metric, symbol Device:C
- added C2: 1u, Capacitor_SMD:C_0402_1005Metric, symbol Device:C
- added C20: 0p8, Capacitor_SMD:C_0402_1005Metric, symbol Device:C
- added C21: 0p3, Capacitor_SMD:C_0402_1005Metric, symbol Device:C
- added D1, D4: LED, LED_SMD:LED_0402_1005Metric, symbol Device:LED
- added D2, D3: PMEG2010AEH, Diode_SMD:D_SOD-123, symbol Device:D_Schottky
- added ENC1, ENC2, ENC3: PEC11R-4220F-S0024, PEC11R_Encoder:Bourns-PEC11R-4220F-S0024-0-0-0, symbol Device:RotaryEncoder_Switch
- added FLT1: DLF162500LT-5028A1, ProdDeck_PCBlib:DLF162500LT-5028A1, symbol ProdDeck_SchemLib:DLF162500LT-5028A1
- added FM1, FM2, FM3: Fiducial, Fiducial:Fiducial_1mm_Mask2mm, symbol Mechanical:Fiducial
- added H1, H3, H4, H5: MountingHole_Pad, MountingHole:MountingHole_3.2mm_M3_Pad, symbol Mechanical:MountingHole_Pad
- added L1: 10n, Inductor_SMD:L_0402_1005Metric, symbol Device:L
- added L2: 10u, Inductor_SMD:L_0805_2012Metric, symbol Device:L
- added L3: 2n7, Inductor_SMD:L_0402_1005Metric, symbol Device:L
- added NRST1: NRST, Button_Switch_SMD:SW_SPST_CK_RS282G05A3, symbol Switch:SW_Push
- added PWR1: Power_Switch, Button_Switch_THT:SW_Slide_SPDT_Straight_CK_OS102011MS2Q, symbol Switch:SW_SPST
- added R1, R10, R2, R3, R4: 5k1, Resistor_SMD:R_0402_1005Metric, symbol Device:R
- added R11: 220R, Resistor_SMD:R_0402_1005Metric, symbol Device:R
- added R12: PTA6043-2015DPB103, slider:POT_PTA6043, symbol slider:PTA6043-2015DPB103
- added R7: 1k, Resistor_SMD:R_0402_1005Metric, symbol Device:R
- added R8, R9: 100k, Resistor_SMD:R_0402_1005Metric, symbol Device:R
- added RF1: Conn_Coaxial, Connector_Coaxial:U.FL_Hirose_U.FL-R-SMT-1_Vertical, symbol Connector:Conn_Coaxial
- added SW3: KEY1, Gateron_KS33_Solderable:Gateron-KS33-Solderable-1U, symbol Switch:SW_Push
- added SW4: KEY4, Gateron_KS33_Solderable:Gateron-KS33-Solderable-1U, symbol Switch:SW_Push
- added SW5: KEY2, Gateron_KS33_Solderable:Gateron-KS33-Solderable-1U, symbol Switch:SW_Push
- added SW6: KEY5, Gateron_KS33_Solderable:Gateron-KS33-Solderable-1U, symbol Switch:SW_Push
- added SW7: KEY3, Gateron_KS33_Solderable:Gateron-KS33-Solderable-1U, symbol Switch:SW_Push
- added SW8: KEY6, Gateron_KS33_Solderable:Gateron-KS33-Solderable-1U, symbol Switch:SW_Push
- added SWD1: TC2030, Connector:Tag-Connect_TC2030-IDC-FP_2x03_P1.27mm_Vertical, symbol Connector:Conn_ARM_SWD_TagConnect_TC2030
- added U1: MIC5365-3.3YD5, Package_TO_SOT_SMD:TSOT-23-5, symbol Regulator_Linear:MIC5365-3.3YD5
- added U2: USBLC6-2SC6, Package_TO_SOT_SMD:SOT-23-6, symbol Power_Protection:USBLC6-2SC6
- added U3: MCP73831-2-OT, Package_TO_SOT_SMD:SOT-23-5, symbol Battery_Management:MCP73831-2-OT
- added U4: STM32WB55CGU6, Package_DFN_QFN:QFN-48-1EP_7x7mm_P0.5mm_EP5.6x5.6mm, symbol MCU_ST_STM32WB:STM32WB55CGUx
- added USB1: USB_C_Receptacle_USB2.0_16P, Connector_USB:USB_C_Receptacle_GCT_USB4105-xx-A_16P_TopMnt_Horizontal, symbol Connector:USB_C_Receptacle_USB2.0_16P
- added X1: 32kHz768, Crystal:Crystal_SMD_2012-2Pin_2.0x1.2mm, symbol Device:Crystal
- added X2: 32MHz, Crystal:Crystal_SMD_2016-4Pin_2.0x1.6mm, symbol Device:Crystal_GND24
Connections:
- new net: D4.1 (K), R7.1
- new net: R7.2, U3.1 (STAT)
- new net: BATT_CONN1.1 (Pin_1), BT1.1 (+), C5.1, PWR1.1 (A), U3.3 (V_{BAT})
- new net: R2.1, USB1.A5 (CC1)
- new net: U2.3 (I/O2), USB1.A6 (D+), USB1.B6 (D+)
- new net: U2.1 (I/O1), USB1.A7 (D-), USB1.B7 (D-)
- new net: R1.1, USB1.B5 (CC2)
- new net: R4.2, U3.5 (PROG)
- new net: BOOT0.1, R11.2
- new net: C1.1, D2.1 (K), D3.1 (K), U1.1 (VIN), U1.3 (EN)
- new net: D2.2 (A), PWR1.2 (B), R8.1
- new net: D1.1 (K), R3.1
- new net +3.3V: BOOT0.2, C10.1, C11.1, C12.1, C13.1, C14.1, C3.1, C4.1, C6.1, C7.1, C8.1, C9.1, D1.2 (A), R12.1, SWD1.1 (VCC), U1.5 (VOUT), U4.1 (VBAT), U4.20 (VDD), U4.23 (VDDRF), U4.34 (VDDSMPS), U4.35 (VDD), U4.40 (VDDUSB), U4.48 (VDD), U4.8 (VDDA)
- new net +5V: C2.1, D3.2 (A), D4.2 (A), U2.5 (VBUS), U3.4 (V_{DD}), USB1.A4 (VBUS), USB1.A9 (VBUS), USB1.B4 (VBUS), USB1.B9 (VBUS)
- new net BATT_SENSE: C15.1, R8.2, R9.1, U4.9 (PA0)
- new net BOOT0: C22.1, R10.1, R11.1, U4.4 (PH3)
- new net ENC1_A: ENC1.A, U4.11 (PA2)
- new net ENC1_B: ENC1.B, U4.12 (PA3)
- new net ENC1_SW: ENC1.S1, U4.19 (PB2)
- new net ENC2_A: ENC2.A, U4.15 (PA6)
- new net ENC2_B: ENC2.B, U4.16 (PA7)
- new net ENC2_SW: ENC2.S1, U4.44 (PB4)
- new net ENC3_A: ENC3.A, U4.28 (PB0)
- new net ENC3_B: ENC3.B, U4.29 (PB1)
- new net ENC3_SW: ENC3.S1, U4.45 (PB5)
- new net GND: BATT_CONN1.2 (Pin_2), BT1.2 (-), C1.2, C10.2, C11.2, C12.2, C13.2, C14.2, C15.2, C16.2, C17.2, C18.2, C19.2, C2.2, C20.2, C21.2, C22.2, C3.2, C4.2, C5.2, C6.2, C7.2, C8.2, C9.2, ENC1.C, ENC1.S2, ENC2.C, ENC2.S2, ENC3.C, ENC3.S2, FLT1.2 (GND), FLT1.4 (GND), H1.1, H3.1, H4.1, H5.1, NRST1.1, R1.2, R10.2, R12.3, R2.2, R3.2, R4.1, R9.2, RF1.2 (Ext), SW3.1, SW4.1, SW5.1, SW6.1, SW7.1, SW8.1, SWD1.5 (GND), U1.2 (GND), U2.2 (GND), U3.2 (V_{SS}), U4.22 (VSSRF), U4.32 (VSSSMPS), U4.49 (VSS), USB1.A1 (GND), USB1.A12 (GND), USB1.B1 (GND), USB1.B12 (GND), USB1.SH (SHIELD), X2.2 (G), X2.4 (G)
- new net HSE_IN: U4.25 (OSC_IN), X2.3
- new net HSE_OUT: U4.24 (OSC_OUT), X2.1
- new net KEY1: SW3.2, U4.13 (PA4)
- new net KEY2: SW5.2, U4.14 (PA5)
- new net KEY3: SW7.2, U4.17 (PA8)
- new net KEY4: SW4.2, U4.18 (PA9)
- new net KEY5: SW6.2, U4.36 (PA10)
- new net KEY6: SW8.2, U4.42 (PA15)
- new net LSE_IN: C17.1, U4.2 (PC14), X1.2
- new net LSE_OUT: C16.1, U4.3 (PC15), X1.1
- new net RF: C20.1, L3.1, U4.21 (RF1)
- new net RF_ANT: FLT1.3 (OUT), RF1.1 (In)
- new net RF_MATCH: C21.1, FLT1.1 (IN), L3.2
- new net SLIDER_WIPER: R12.2, U4.10 (PA1)
- new net SMPSFB: C19.1, L2.2, U4.31 (VFBSMPS)
- new net SMPSLX: L1.1, U4.33 (VLXSMPS)
- new net SMPSLXL: L1.2, L2.1
- new net SWD_CLK: SWD1.4 (SWCLK), U4.41 (PA14)
- new net SWD_DIO: SWD1.2 (SWDIO), U4.39 (PA13)
- new net SWD_NRST: C18.1, NRST1.2, SWD1.3 (~{RESET}), U4.7 (NRST)
- new net SWD_TRC: SWD1.6 (SWO), U4.43 (PB3)
- new net USB_D+: U2.4 (I/O2), U4.38 (PA12)
- new net USB_D-: U2.6 (I/O1), U4.37 (PA11)
- no-connect marks 0 -> 7
Other:
- note added: "BOOT0 Switch"
- note added: "Buttons + Slider"
- note added: "LSH and HSE"
- note added: "LiPo Battery Charging Module"
- note added: "RF Front-End & u.FL Connector"
- note added: "Rotary Encoders"
- note added: "STM32 MCU"
- note added: "Voltage Regulator (down to 3.3v)"
- title: (none) -> ProdDeck Schematic

Commit message: pcb done
Parts:
- BATT_CONN1, ENC1, ENC2, ENC3, PWR1, R12, SW3, SW4, SW5, SW6, SW7, SW8: now fitted
Changed lines of the file:
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@@
 		(on_board yes)
 		(in_pos_files yes)
-		(dnp yes)
+		(dnp no)
 		(property "Reference" "SW6"
 			(at 212.09 153.75 0)
@@
 		(on_board yes)
 		(in_pos_files yes)
-		(dnp yes)
+		(dnp no)
 		(property "Reference" "BATT_CONN1"
 			(at 39.37 157.734 0)
@@
 		(on_board yes)
 		(in_pos_files yes)
-		(dnp yes)
+		(dnp no)
 		(property "Reference" "R12"
 			(at 268.478 153.924 90)
@@
 		(on_board yes)
 		(in_pos_files yes)
-		(dnp yes)
+		(dnp no)
 		(property "Reference" "SW5"
 			(at 212.09 139.78 0)
@@
 		(on_board yes)
 		(in_pos_files yes)
-		(dnp yes)
+		(dnp no)
 		(property "Reference" "ENC1"
 			(at 180.086 27.94 0)
@@
 		(on_board yes)
 		(in_pos_files yes)
-		(dnp yes)
+		(dnp no)
 		(property "Reference" "SW3"
 			(at 189.23 139.78 0)
@@
 		(on_board yes)
 		(in_pos_files yes)
-		(dnp yes)
+		(dnp no)
 		(property "Reference" "SW4"
 			(at 189.23 153.75 0)
@@
 		(on_board yes)
 		(in_pos_files yes)
-		(dnp yes)
+		(dnp no)
 		(property "Reference" "SW7"
 			(at 236.22 139.78 0)
@@
 		(on_board yes)
 		(in_pos_files yes)
-		(dnp yes)
+		(dnp no)
 		(property "Reference" "PWR1"
 			(at 78.74 180.42 0)
@@
 		(on_board yes)
 		(in_pos_files yes)
-		(dnp yes)
+		(dnp no)
 		(property "Reference" "SW8"
 			(at 236.22 153.75 0)
@@
 		(on_board yes)
 		(in_pos_files yes)
-		(dnp yes)
+		(dnp no)
 		(property "Reference" "ENC3"
 			(at 261.62 27.686 0)
@@
 		(on_board yes)
 		(in_pos_files yes)
-		(dnp yes)
+		(dnp no)
 		(property "Reference" "ENC2"
 			(at 220.98 27.432 0)
